File: hardware/shield-PCB/Shield1.brd (EAGLE design)
At the start: 160 x 100 mm, 107 parts, among them IC1 74LVC1G125DBV, IC11 KNOCK_SENS_IC_TPIC8101, IC2 74LVC1G125DBV, IC3 74LVC1G125DBV, IC4 MC33269ST-3.3T3, IC5 74LVC1G125DBV, IC6 MC33810SSOP, IC7 MCP6561U-SOT23, IC8 AP1117(5V), IC9 MC33269-5V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

Commit message: Update schematic to show tach power and pullup
Parts:
- added OK1: 4N33, optocoupler:DIL06
- added R33: 10k, rcl:R1206
Connections:
- removed net N$5: FUSE1.1, U$1.19
- new net AIR_V+: FUSE1.1, OK1.6, U$1.19
- net +5V: now also R33.1
- net GND: now also OK1.4
- net TACH: now also OK1.5, R33.2
Routing:
- net N$5: track 6.39 -> 0.00 mm
- net AIR_V+: track 0.00 -> 6.39 mm
Changed lines of the file:
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@@
 <layer number="2" name="Route2" color="1" fill="3" visible="no" active="no"/>
 <layer number="3" name="Route3" color="4" fill="3" visible="no" active="no"/>
+<layer number="4" name="Route4" color="1" fill="4" visible="no" active="no"/>
+<layer number="5" name="Route5" color="4" fill="4" visible="no" active="no"/>
+<layer number="6" name="Route6" color="1" fill="8" visible="no" active="no"/>
+<layer number="7" name="Route7" color="4" fill="8" visible="no" active="no"/>
+<layer number="8" name="Route8" color="1" fill="2" visible="no" active="no"/>
+<layer number="9" name="Route9" color="4" fill="2" visible="no" active="no"/>
+<layer number="10" name="Route10" color="1" fill="7" visible="no" active="no"/>
+<layer number="11" name="Route11" color="4" fill="7" visible="no" active="no"/>
+<layer number="12" name="Route12" color="1" fill="5" visible="no" active="no"/>
+<layer number="13" name="Route13" color="4" fill="5" visible="no" active="no"/>
 <layer number="14" name="Route14" color="1" fill="6" visible="no" active="no"/>
 <layer number="15" name="Route15" color="4" fill="6" visible="no" active="no"/>
@@
 <element name="JP8" library="pinhead" package="1X05" value="" x="64.135" y="96.52" rot="R180"/>
 <element name="R26" library="rcl" package="R1206" value="22k" x="20.955" y="40.64" rot="R270"/>
+<element name="OK1" library="optocoupler" package="DIL06" value="4N33" x="-13.97" y="-9.525">
+<attribute name="OC_NEWARK" value="88K1390" x="-13.97" y="-9.525" size="1.778" layer="27" display="off"/>
+<attribute name="MPN" value="4N33" x="-13.97" y="-9.525" size="1.778" layer="27" display="off"/>
+<attribute name="MF" value="VISHAY/TELEFUNKEN" x="-13.97" y="-9.525" size="1.778" layer="27" display="off"/>
+<attribute name="OC_FARNELL" value="1469601" x="-13.97" y="-9.525" size="1.778" layer="27" display="off"/>
+</element>
+<element name="R33" library="rcl" package="R1206" value="10k" x="-17.145" y="-19.685"/>
 </elements>
 <signals>
@@
 <contactref element="R26" pad="2"/>
 <contactref element="U$1" pad="17"/>
+<contactref element="OK1" pad="4"/>
+<wire x1="103.505" y1="97.79" x2="105.41" y2="97.79" width="0" layer="19" extent="1-1"/>
+<wire x1="101.6" y1="97.79" x2="103.505" y2="97.79" width="0" layer="19" extent="1-1"/>
+<wire x1="110.49" y1="87.478" x2="105.41" y2="97.79" width="0" layer="19" extent="1-1"/>
+<wire x1="111.125" y1="78.257" x2="110.49" y2="87.478" width="0" layer="19" extent="1-1"/>
+<wire x1="104.4575" y1="69.5325" x2="111.125" y2="78.257" width="0" layer="19" extent="1-1"/>
+<wire x1="78.46" y1="71.475" x2="81.635" y2="71.475" width="0" layer="19" extent="1-1"/>
+<wire x1="111.125" y1="54.458" x2="108.9025" y2="65.405" width="0" layer="19" extent="1-1"/>
+<wire x1="111.125" y1="45.237" x2="111.125" y2="54.458" width="0" layer="19" extent="1-1"/>
+<wire x1="71.625" y1="52.705" x2="75.535" y2="67.9" width="0" layer="19" extent="1-1"/>
+<wire x1="110.805" y1="29.23" x2="111.125" y2="45.237" width="0" layer="19" extent="1-1"/>
+<wire x1="71.12" y1="32.255" x2="69.85" y2="48.895" width="0" layer="19" extent="1-1"/>
+<wire x1="64.265" y1="30.48" x2="71.12" y2="32.255" width="0" layer="19" extent="1-1"/>
+<wire x1="62.865" y1="21.336" x2="64.265" y2="30.48" width="0" layer="19" extent="1-1"/>
+<wire x1="78.105" y1="8.76" x2="74.295" y2="13.335" width="0" layer="19" extent="1-1"/>
+<wire x1="54.965" y1="8.515" x2="61.965" y2="12.565" width="0" layer="19" extent="1-1"/>
+<wire x1="65.615" y1="4.84" x2="62.29" y2="12.565" width="0" layer="19" extent="1-1"/>
+<wire x1="50.673" y1="33.02" x2="64.265" y2="30.48" width="0" layer="19" extent="1-1"/>
+<wire x1="47.117" y1="30.48" x2="50.673" y2="33.02" width="0" layer="19" extent="1-1"/>
+<wire x1="43.18" y1="17.78" x2="47.117" y2="30.48" width="0" layer="19" extent="1-1"/>
+<wire x1="43.18" y1="15.875" x2="43.18" y2="17.78" width="0" layer="19" extent="1-1"/>
+<wire x1="39.37" y1="15.875" x2="43.18" y2="15.875" width="0" layer="19" extent="1-1"/>
+<wire x1="34.925" y1="5.715" x2="39.37" y2="13.465" width="0" layer="19" extent="1-1"/>
+<wire x1="29.845" y1="8.255" x2="34.925" y2="5.715" width="0" layer="19" extent="1-1"/>
+<wire x1="27.516" y1="23.556" x2="35.9664" y2="18.3388" width="0" layer="19" extent="1-1"/>
+<wire x1="27.305" y1="27.305" x2="27.516" y2="23.556" width="0" layer="19" extent="1-1"/>
+<wire x1="29.845" y1="27.305" x2="27.305" y2="27.305" width="0" layer="19" extent="1-1"/>
+<wire x1="27.5336" y1="31.75" x2="27.305" y2="27.305" width="0" layer="19" extent="1-1"/>
+<wire x1="24.765" y1="33.525" x2="27.5336" y2="32.4612" width="0" layer="19" extent="1-1"/>
+<wire x1="33.15" y1="36.325" x2="27.5336" y2="32.4612" width="0" layer="19" extent="1-1"/>
+<wire x1="20.955" y1="39.218" x2="24.765" y2="33.525" width="0" layer="19" extent="1-1"/>
+<wire x1="18.415" y1="38.74" x2="20.955" y2="39.218" width="0" layer="19" extent="1-1"/>
+<wire x1="15.24" y1="39.24" x2="18.415" y2="38.74" width="0" layer="19" extent="1-1"/>
+<wire x1="15.875" y1="49.025" x2="15.24" y2="39.24" width="0" layer="19" extent="1-1"/>
+<wire x1="4" y1="51.5" x2="12.7" y2="49.525" width="0" layer="19" extent="1-1"/>
+<wire x1="4" y1="46.5" x2="4" y2="51.5" width="0" layer="19" extent="1-1"/>
+<wire x1="9" y1="59" x2="4" y2="51.5" width="0" layer="19" extent="1-1"/>
+<wire x1="25.146" y1="83.185" x2="24.765" y2="73.66" width="0" layer="19" extent="1-1"/>
+<wire x1="22.86" y1="84.585" x2="25.146" y2="83.185" width="0" layer="19" extent="1-1"/>
+<wire x1="20.32" y1="84.885" x2="22.86" y2="84.585" width="0" layer="19" extent="1-1"/>
+<wire x1="114.3" y1="8.255" x2="111.76" y2="27.94" width="0" layer="19" extent="1-1"/>
+<wire x1="104.57" y1="8.145" x2="114.3" y2="8.255" width="0" layer="19" extent="1-1"/>
+<wire x1="-11.43" y1="-5.715" x2="27.305" y2="5.715" width="0" layer="19" extent="1-1"/>
 </signal>
 <signal name="N$1">
@@
 <wire x1="35.56" y1="46.99" x2="34.29" y2="46.99" width="0.6096" layer="1"/>
 <wire x1="34.29" y1="46.99" x2="31.75" y2="44.45" width="0.6096" layer="1"/>
+<contactref element="R33" pad="1"/>
+<wire x1="31.75" y1="42.545" x2="31.75" y2="44.45" width="0" layer="19" extent="1-1"/>
+<wire x1="29.845" y1="44.45" x2="31.75" y2="44.45" width="0" layer="19" extent="1-1"/>
+<wire x1="27.94" y1="44.45" x2="29.845" y2="44.45" width="0" layer="19" extent="1-1"/>
+<wire x1="27.94" y1="42.545" x2="29.845" y2="42.545" width="0" layer="19" extent="16-16"/>
+<wire x1="-18.567" y1="-19.685" x2="32.385" y2="27.305" width="0" layer="19" extent="1-1"/>
 </signal>
 <signal name="SEL3">
@@
 <contactref element="U$1" pad="1"/>
 <wire x1="4.11" y1="76.5" x2="4" y2="76.5" width="0.4064" layer="1"/>
+<contactref element="OK1" pad="5"/>
+<contactref element="R33" pad="2"/>
+<wire x1="-13.97" y1="-5.715" x2="4" y2="76.5" width="0" layer="19" extent="1-1"/>
+<wire x1="-15.723" y1="-19.685" x2="-13.97" y2="-5.715" width="0" layer="19" extent="1-1"/>
 </signal>
 <signal name="N$11">
@@
 <wire x1="95.0595" y1="75.8825" x2="95.377" y2="76.2" width="0.3048" layer="1"/>
 </signal>
-<signal name="N$5">
-<contactref element="U$1" pad="19"/>
-<contactref element="FUSE1" pad="1"/>
-<wire x1="13.106" y1="52.705" x2="11.43" y2="52.705" width="0.4064" layer="1"/>
-<wire x1="11.43" y1="52.705" x2="9.525" y2="50.8" width="0.4064" layer="1"/>
-<wire x1="9.525" y1="50.8" x2="9.525" y2="49.525" width="0.4064" layer="1"/>
-<wire x1="9.525" y1="49.525" x2="9" y2="49" width="0.4064" layer="1"/>
-</signal>
 <signal name="O2_SENS">
 <contactref element="U$1" pad="5"/>
@@
 <wire x1="56.515" y1="93.98" x2="56.515" y2="87.884" width="0.4064" layer="1"/>
 </signal>
+<signal name="AIR_V+">
+<contactref element="OK1" pad="6"/>
+<contactref element="U$1" pad="19"/>
+<contactref element="FUSE1" pad="1"/>
+<wire x1="13.106" y1="52.705" x2="11.43" y2="52.705" width="0.4064" layer="1"/>
+<wire x1="11.43" y1="52.705" x2="9.525" y2="50.8" width="0.4064" layer="1"/>
+<wire x1="9.525" y1="50.8" x2="9.525" y2="49.525" width="0.4064" layer="1"/>
+<wire x1="9.525" y1="49.525" x2="9" y2="49" width="0.4064" layer="1"/>
+<wire x1="-16.51" y1="-5.715" x2="9" y2="49" width="0" layer="19" extent="1-1"/>
+</signal>
 </signals>
